File: pcb/usb_a.kicad_sch (KiCad schematic)
At the start: 3 parts, among them U1 NDP5102SE, U2 USBLC6-4SC6-ES

Commit message: finished schematic and pcb woohoo!
Parts:
- removed U2: USBLC6-4SC6-ES, easyeda2kicad:SOT-23-6_L2.9-W1.6-P0.95-LS2.8-BL, symbol easyeda2kicad:USBLC6-4SC6-ES
- added C1: 100n, Capacitor_SMD:C_0603_1608Metric, symbol Device:C
- added U18: USBLC6-4SC6, Package_TO_SOT_SMD:SOT-23-6, symbol Power_Protection:USBLC6-4SC6
- U3: renamed from U1; MPN (none) -> NDP5102SE; Manufacturer (none) -> NDP(芯潭微)
- USB1: MPN (none) -> AF SS-JB17.6; Manufacturer (none) -> SHOU HAN(首韩)
Connections:
- net GND: now also U3.2 (GND), USB1.10 (SHELL), USB1.11 (SHELL), USB1.12 (SHELL), USB1.9 (SHELL), C1.2, U18.2 (GND)
- net 1D+: now reaches U3.1 (DP1)
- net 1D+: now also USB1.3 (D+), U18.3 (I/O2)
- net 2D+: now reaches U3.3 (DP2)
- net 2D+: now also USB1.7 (D+), U18.4 (I/O3)
- net 2D-: now reaches U3.4 (DM2)
- net 2D-: now also USB1.6 (D-), U18.6 (I/O4)
- net +5V: now reaches U3.5 (VCC)
- net +5V: now also USB1.1 (VCC), USB1.5 (VCC), C1.1, U18.5 (VBUS)
- net 1D-: now reaches U3.6 (DM1)
- net 1D-: now also USB1.2 (D-), U18.1 (I/O1)
Other:
- moved on the sheet: U3, USB1
