File: pcb/skibidi-usb-charger-hub.kicad_sch (KiCad schematic)
At the start: 0 parts

Commit message: finished schematic and pcb woohoo!
Parts:
- added H13, H14, H15, H16, H17, H18: MountingHole, MountingHole:MountingHole_3.2mm_M3_Pad, symbol Mechanical:MountingHole
- added H19, H20, H21, H22: MountingHole, extras:ZipTie_Hole, symbol Mechanical:MountingHole
Other:
- sheet 5V USB A renamed 5V USB A 1
- added sheet 5V USB A 2 (usb_a.kicad_sch)
- added sheet 5V USB C (usb_c.kicad_sch)
- added sheet PD USB C 1 (usb_c_pd.kicad_sch)
- added sheet PD USB C 2 (usb_c_pd.kicad_sch)
- added sheet PD USB C 3 (usb_c_pd.kicad_sch)
- added sheet PD USB C 4 (usb_c_pd.kicad_sch)

Commit message: add gerbers
Other:
- company: Toby Cm's Lab -> Toby Cm's Lab x Hack Club
Changed lines of the file:
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@@
 		(date "2026-03-15")
 		(rev "v1")
-		(company "Toby Cm's Lab")
+		(company "Toby Cm's Lab x Hack Club")
 	)
 	(symbol
